File: OpenPilot-PicoCC/ESC-stub.sch (EAGLE design)
At the start: 76 parts, among them U1 STM32F103CBT6, U3 LM4120AIM5-1.8, U4 LT6654AHS6-3.3TRMPBF, U5 L3G4200D, X1 MINI-USB-SCHIELD-32005-301, X2 08FLZ-SM1

Commit message: Updated Readme Some initial ESD Setup
Parts:
- removed C1, C17, C18, C19, C2, C20: (no value), rcl:C-USC0402
- removed C15, C16, C3, C4, C5, C6, C7, C8: (no value), rcl:C-USC0402K
- removed D1: BAT54C, diode:BAT54C
- removed JP10, JP11, JP12, JP7, JP8, JP9: (no value), SparkFun:M03POGO_PIN_HOLES_ONLY
- removed R1, R10, R11, R12, R13, R14, R15, R16, R5, R6, R7, R8, R9: (no value), rcl:R-US_R0402
- removed SJ1: (no value), jumper:SJ2WW
- removed TP1, TP10, TP11, TP2, TP3, TP4, TP5, TP6, TP7, TP8, TP9: TPSQTP12R, testpad:TPSQTP12R
- removed U$1: (no value), TI_TPS:TPS7A6033-Q1
- removed U$10: ADXL345, analog-devices:ADXL345
- removed U$11: S2SFL064K, SPANSION:S2SFL064K
- removed U$12, U$15, U$17, U$3, U$4, U$5, U$6, U$7, U$8: NUP1301, NXP:NUP1301
- removed U$13: ABM3B, ABRACON:ABM3B
- removed U$2: T495-8528-21, Kemet:T495-8528-21
- removed U$22: PRTR5V0U2D, NXP:PRTR5V0U2D
- removed U$9: PCS3P258XX, on-semiconductor:PCS3P258XX
- removed U1: STM32F103CBT6, st-microelectronics:STM32F103CBT6
- removed U3: LM4120AIM5-1.8, national-semiconductor:LM4120AIM5-1.8
- removed U4: LT6654AHS6-3.3TRMPBF, linear-technology:LT6654AHS6-3.3TRMPBF
- removed U5: L3G4200D, SparkFun:L3G4200D
- removed X1: MINI-USB-SCHIELD-32005-301, con-cypressindustries:MINI-USB-SCHIELD-32005-301
- removed X2: 08FLZ-SM1, con-jst:08FLZ-SM1
- added C10, C11, C12, C13, C14, C9: (no value), rcl:C-USC0402K
- added D2, D3, D4, D5, D6, D7: BAS40-05, diode:BAS40-05
- added PAD1, PAD2, PAD3: WIREPADSMD5-2,5, wirepad:WIREPADSMD5-2,5
- added U$19: 2PC4617, NXP:2PC4617
- R2, R3, R4: device rcl:R-US_R0402 -> rcl:R-US_R2512W
- U$14, U$16, U$18: value NUP1301 -> IRF7309Q; device NXP:NUP1301 -> IR-HEXFET:IRF7309Q
- U$20: value PRTR5V0U4D -> 2PC4617; device NXP:PRTR5V0U4D -> NXP:2PC4617
- U$21: value PRTR5V0U2D -> 2PC4617; device NXP:PRTR5V0U2D -> NXP:2PC4617
Connections:
- removed net 3.3V: C1.1, C15.1, C17.1, C18.1, C2.1, C7.1, C8.1, R1.2, R5.2, R6.2, TP4.TP, U$1.VOUT, U$10.RES-VS, U$10.VS, U$11.HOLD_(IO3), U$11.VCC, U$11.WP_(IO2), U$9.VDD, U1.VBAT, U1.VDD_1, U1.VDD_2, U1.VDD_3, U3.EN, U3.VIN, U5.RSVDV@0, U5.VDD, U5.VDDIO
- removed net AGND: C3.1, C4.2, JP10.3, JP11.3, JP12.3, JP7.3, JP8.3, JP9.3, SJ1.1, TP1.TP, U$1.GND, U$1.GND_T, U$12.1, U$14.1, U$15.1, U$16.1, U$17.1, U$18.1, U$2.2, U$3.1, U$4.1, U$5.1, U$6.1, U$7.1, U$8.1, X2-1.1
- removed net DGND: C1.2, C15.2, C16.2, C17.2, C18.2, C19.1, C2.2, C5.2, C6.2, C7.2, C8.2, R7.2, SJ1.3, TP2.TP, U$10.GND2, U$10.GND4, U$10.GND5, U$10.RES-GND, U$11.GND, U$13.GND1, U$13.GND2, U$9.FSEL, U$9.S0, U$9.VSS, U3.GND, U5.GND, U5.RSDVG@3, U5.RSVDG@0, U5.RSVDG@1, U5.RSVDG@2, U5.RSVDG@4
- removed net N$1: R16.2, R2.1, U$12.3
- removed net N$10: JP9.1, TP7.TP, U$5.3, U1.PA8
- removed net N$11: JP10.1, TP8.TP, U$6.3, U1.PB7
- removed net N$12: JP11.1, TP9.TP, U$7.3, U1.PB8
- removed net N$13: JP12.1, TP10.TP, U$8.3, U1.PB9
- removed net N$14: TP11.TP, U$9.MODOUT, U1.PD0-OSC_IN
- removed net N$15: R5.1, U$11.CS, U1.PA7
- removed net N$16: U$11.CLK, U1.PB13
- removed net N$17: U$10.SDA, U$11.SI_(IO0), U1.PB15
- removed net N$18: U$10.SDO, U$11.SO_(IO1), U1.PB14
- removed net N$2: U1.PA11
- removed net N$3: C4.1, D1.CC, TP3.TP, U$1.VIN, U$2.1
- removed net N$37: C6.1, U$13.CR2, U$9.XOUT
- removed net N$38: C5.1, U$13.CR1, U$9.XIN
- removed net N$4: C3.2, U$1.RDELAY
- removed net N$40: U$10.INT1, U1.PC14-OSC32_IN
- removed net N$41: U$10.INT2, U1.PC13-TAMPER-RTC
- removed net N$43: R6.1, U$10.!CS, U1.PB12
- removed net N$46: C20.1, R7.1
- removed net N$47: C19.2, C20.2, U5.PLL
- removed net N$5: U$22.4, U1.PA12
- removed net N$6: R1.1, U$1.NRST
- removed net N$7: U$22.6
- removed net N$8: JP7.1, TP5.TP, U$3.3, U1.PA2
- removed net N$9: JP8.1, TP6.TP, U$4.3, U1.PB4
- removed net VCC: D1.A1, JP10.2, JP11.2, JP12.2, JP7.2, JP8.2, JP9.2, U$12.2, U$14.2, U$15.2, U$16.2, U$17.2, U$18.2, U$3.2, U$4.2, U$5.2, U$6.2, U$7.2, U$8.2, X2-2.1
- removed net VEE: C16.1, U3.VOUT
- new net N$36: C11.2, C12.2, D4.A1, D4.C, D5.A1, R3.2, U$16.N-D$1, U$16.N-D$2, U$16.P-D$1, U$16.P-D$2
- net N$19: now also U$14.P-G, U$19.P$3; no longer R2.2, X2-8.1
- net N$20: now also U$14.N-G; no longer R15.2, R3.1, U$14.3
- net N$21: now also U$18.N-G; no longer R14.2, R4.1, U$15.3
- net N$22: now also U$16.P-G, U$20.P$3; no longer R8.2, X2-5.1
- net N$23: now also U$16.N-G; no longer R3.2, X2-7.1
- net N$24: now also U$18.P-G, U$21.P$3; no longer R10.2, X2-3.1
- net N$25: now also C10.2, C9.2, D2.A1, D2.C, D3.A1, R2.1, U$14.N-D$1, U$14.N-D$2, U$14.P-D$1, U$14.P-D$2; no longer R9.2, X2-4.1
- net N$26: now also PAD1.P, R2.2; no longer R13.2, R8.1, U$16.3
- net N$27: now also PAD2.P, R3.1; no longer R12.2, R9.1, U$17.3
- net N$28: now also PAD3.P, R4.2; no longer R10.1, R11.2, U$18.3
- net N$29: now also C9.1, D2.A2, U$14.N-S; no longer R4.2, X2-6.1
- net N$30: now also C10.1, D3.A2, D3.C, U$14.P-S; no longer R16.1, U1.PA1
- net N$31: now also C13.1, D6.A2, U$18.N-S; no longer R15.1, U1.PA0-WKUP
- net N$32: now also C14.1, D7.A2, D7.C, U$18.P-S; no longer R14.1, U1.PB1
- net N$33: now also C11.1, D4.A2, U$16.N-S; no longer R13.1, U1.PB0
- net N$34: now also C12.1, D5.A2, D5.C, U$16.P-S; no longer R12.1, U1.PB5
- net N$35: now also C13.2, C14.2, D6.A1, D6.C, D7.A1, R4.1, U$18.N-D$1, U$18.N-D$2, U$18.P-D$1, U$18.P-D$2; no longer R11.1, U1.PB6
Other:
- note added: "M"
- note added: "Source"
- moved on the sheet: R2, R3, R4
