File: OpenPilot-PicoCC/PicoCC.sch (EAGLE design)
At the start: 97 parts, among them U5 L3G4200D, X1 MINI-USB-SCHIELD-32005-301, X2 08FLZ-SM1

Commit message: Initial Power Level Test Layout, might be able to do under 3cm
Parts:
- added C12, C13: (no value), rcl:C-USC0402
- added SJ4: (no value), jumper:SJ2W
Connections:
- new net N$20: C13.1, SJ4.3, U$16.VSS_1
- new net N$3: C12.1, SJ4.2, U$16.VSS_2
- net DGND: now also C12.2, C13.2, SJ4.1
Other:
- note added: "F2-F4 Bypass"
- moved on the sheet: C15, C17, C18, C19, C20, R5, R6, R7, SJ3, TP20, TP21, TP22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
