File: OpenPilot-PicoCC/PowerLevel.sch (EAGLE design)
At the start: 97 parts, among them U1 STM32F103CBT6, U5 L3G4200D, X1 MINI-USB-SCHIELD-32005-301, X2 08FLZ-SM1

Commit message: Initial Power Level Test Layout, might be able to do under 3cm
Parts:
- removed C15, C5, C6, C7, C8: (no value), rcl:C-USC0402K
- removed C17, C18, C19, C20: (no value), rcl:C-USC0402
- removed JP10, JP11, JP12, JP7, JP8, JP9: (no value), SparkFun:M03POGO_PIN_HOLES_ONLY
- removed L1: BML15HB121SN1, inductors:BML15HB121SN1
- removed R10, R11, R12, R13, R14, R15, R16, R17, R18, R19, R2, R3, R4, R5, R6, R7, R8, R9: (no value), rcl:R-US_R0402
- removed SJ2, SJ3: (no value), jumper:SJ2WW
- removed TP1, TP10, TP11, TP12, TP13, TP14, TP15, TP16, TP17, TP18, TP19, TP2, TP20, TP21, TP22, TP23, TP24, TP25, TP26, TP27, TP28, TP29, TP3, TP4, TP5, TP6, TP7, TP8, TP9: TPSQTP12R, testpad:TPSQTP12R
- removed U$10: ADXL345, analog-devices:ADXL345
- removed U$11: S2SFL064K, SPANSION:S2SFL064K
- removed U$13: ABM3B, ABRACON:ABM3B
- removed U$19, U$20: PRTR5V0U4D, NXP:PRTR5V0U4D
- removed U$21: PRTR5V0U2D, NXP:PRTR5V0U2D
- removed U$3, U$4, U$5, U$6, U$7, U$8: NUP1301, NXP:NUP1301
- removed U$9: PCS3P258XX, on-semiconductor:PCS3P258XX
- removed U1: STM32F103CBT6, st-microelectronics:STM32F103CBT6
- removed U5: L3G4200D, SparkFun:L3G4200D
- removed X1: MINI-USB-SCHIELD-32005-301, con-cypressindustries:MINI-USB-SCHIELD-32005-301
- removed X2: 08FLZ-SM1, con-jst:08FLZ-SM1
- added !RESET, !RESET_S, 3.3V, 3.3V_S, AGND, DGND, VBAT, VBAT2, VBUS, VDD: (no value), pinhead:PINHD-1X1
- C1, C4, C9: value (none) -> 0.1uF
- C10, C2: value (none) -> 10uF
- C11, C3: value (none) -> 100pF
- R1, R20: value (none) -> 1k
Connections:
- removed net 3.3V: C1.1, C15.1, C17.1, C18.1, C2.1, C7.1, C8.1, R1.2, R15.2, R3.1, R5.2, R6.2, TP4.TP, U$1.VOUT, U$10.RES-VS, U$10.VS, U$11.HOLD_(IO3), U$11.VCC, U$11.WP_(IO2), U$19.5, U$20.6, U$9.VDD, U1.VBAT, U1.VDD_1, U1.VDD_2, U1.VDD_3, U5.RSVDV@0, U5.VDD, U5.VDDIO
- removed net D+: R17.2, U$19.4, X1G$1.2
- removed net D+2: R17.1, TP18.TP, U1.PA11
- removed net D-: R18.2, U$19.6, X1G$1.3
- removed net D-2: R18.1, R19.1, TP19.TP, U1.PA12
- removed net N$10: JP9.1, TP7.TP, U$5.3, U1.PA8
- removed net N$11: JP10.1, TP8.TP, U$6.3, U1.PB7
- removed net N$12: JP11.1, TP9.TP, U$7.3, U1.PB8
- removed net N$13: JP12.1, TP10.TP, U$8.3, U1.PB9
- removed net N$14: TP11.TP, U$9.MODOUT, U1.PD0-OSC_IN
- removed net N$15: R5.1, TP23.TP, U$11.CS, U1.PA7
- removed net N$16: TP22.TP, U$11.CLK, U1.PB13
- removed net N$17: TP21.TP, U$10.SDA, U$11.SI_(IO0), U1.PB15
- removed net N$18: TP20.TP, U$10.SDO, U$11.SO_(IO1), U1.PB14
- removed net N$19: R2.2, X2-8.1
- removed net N$22: R8.2, X2-5.1
- removed net N$23: R3.2, X2-7.1
- removed net N$24: R10.2, X2-3.1
- removed net N$25: R9.2, X2-4.1
- removed net N$29: R4.2, X2-6.1
- removed net N$30: R16.1, TP12.TP, U1.PA1
- removed net N$31: R15.1, TP13.TP, U1.PA0-WKUP
- removed net N$32: R14.1, TP14.TP, U1.PB1
- removed net N$33: R13.1, TP15.TP, U1.PB0
- removed net N$34: R12.1, TP16.TP, U1.PB5
- removed net N$35: R11.1, TP17.TP, U1.PB6
- removed net N$36: R16.2, R2.1, U$20.4
- removed net N$37: C6.1, U$13.CR2, U$9.XOUT
- removed net N$38: C5.1, U$13.CR1, U$9.XIN
- removed net N$39: R14.2, R4.1, U$20.1
- removed net N$40: U$10.INT1, U1.PC14-OSC32_IN
- removed net N$41: U$10.INT2, U1.PC13-TAMPER-RTC
- removed net N$42: R13.2, R8.1, U$20.3
- removed net N$43: R6.1, U$10.!CS, U1.PB12
- removed net N$44: R10.1, R11.2, U$19.3
- removed net N$45: R12.2, R9.1, U$19.1
- removed net N$46: C20.1, R7.1
- removed net N$47: C19.2, C20.2, U5.PLL
- removed net N$8: JP7.1, TP5.TP, U$3.3, U1.PA2
- removed net N$9: JP8.1, TP6.TP, U$4.3, U1.PB4
- removed net VCC: D1.A1, D1.A2, JP10.2, JP11.2, JP12.2, JP7.2, JP8.2, JP9.2, L1.2, R19.2, U$3.2, U$4.2, U$5.2, U$6.2, U$7.2, U$8.2, X2-2.1
- removed net VEE: C10.1, C9.1, R20.2, TP29.TP, U$15.VOUT, U1.VDDA
- new net 3.3V_SECONDARY: 3.3V_S.1, C10.1, C9.1, R20.2, U$15.VOUT
- new net N$3: SJ1.2, VDD.1
- new net VBAT: D1.A1, VBAT.1, VBAT2.1
- new net VUSB: D1.A2, VBUS.1
- net AGND: now also AGND.1; no longer JP10.3, JP11.3, JP12.3, JP7.3, JP8.3, JP9.3, SJ2.1, SJ3.1, TP1.TP, TP24.TP, TP26.TP, U$19.2, U$20.2, U$3.1, U$4.1, U$5.1, U$6.1, U$7.1, U$8.1, X1G$1.5, X1S.S1, X1S.S2, X1S.S3, X1S.S4, X2-1.1
- net DGND: now also DGND.1; no longer C15.2, C17.2, C18.2, C19.1, C5.2, C6.2, C7.2, C8.2, R7.2, SJ2.3, SJ3.3, TP2.TP, TP25.TP, TP27.TP, U$10.GND2, U$10.GND4, U$10.GND5, U$10.RES-GND, U$11.GND, U$13.GND1, U$13.GND2, U$9.FSEL, U$9.S0, U$9.VSS, U5.GND, U5.RSDVG@3, U5.RSVDG@0, U5.RSVDG@1, U5.RSVDG@2, U5.RSVDG@4
- net N$1: now also 3.3V.1, C1.1, C2.1, R1.2, U$1.VOUT; no longer L1.1, X1G$1.1
- net N$2: no longer TP28.TP, TP3.TP
- net N$6: now also !RESET.1
- net N$7: now also !RESET_S.1
Other:
- note removed: "Sensor Level"
- note removed: "Temp Range -40C to +85C"
- moved on the sheet: C1, C10, C11, C2, C3, C4, C9, D1, R1, R20, SJ1, U$1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
